File: circuit/eagle/projects/Inverted_Pendulum-in-TAHU/untitled.brd (EAGLE design)
At the start: 16 parts, among them X3 332-02

Commit message: Update circuit
Parts:
- added S3: TL39PO, switch:TL3XPO
- moved C3 60.3 mm to (43.2, 8.89)
- moved C2 48.3 mm to (31.8, 10.2)
- moved DRIVER1 6.35 mm to (11.4, 20.3)
- moved DRIVER2 3.81 mm to (17.8, 36.8)
Connections:
- net N$10: now also C1.1, DRIVER1.8, DRIVER2.8, S3.1, SV1.1; no longer DRIVER1.7, MOTOR1.5, SV1.4
- net N$7: now also DRIVER1.7, MOTOR1.5, SV1.4
- net VCC: now also S3.2; no longer C1.1, DRIVER1.8, DRIVER2.8, SV1.1
Changed lines of the file:
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@@
 </autorouter>
 <elements>
-<element name="DRIVER1" library="TA7291P" package="HSIP10" value="TA7291" x="15.24" y="25.4"/>
-<element name="DRIVER2" library="TA7291P" package="HSIP10" value="TA7291" x="13.97" y="36.83"/>
+<element name="DRIVER1" library="TA7291P" package="HSIP10" value="TA7291" x="11.43" y="20.32"/>
+<element name="DRIVER2" library="TA7291P" package="HSIP10" value="TA7291" x="17.78" y="36.83"/>
 <element name="SV1" library="con-lstb" package="MA08-1" value="" x="11.43" y="2.54">
 <attribute name="OC_FARNELL" value="unknown" x="11.43" y="2.54" size="1.778" layer="27" display="off"/>
@@
 <attribute name="OC_NEWARK" value="unknown" x="58.42" y="21.59" size="1.778" layer="27" display="off"/>
 </element>
-<element name="C2" library="capacitor-wima" package="C5B2.5" value="0.1uF" x="3.81" y="-29.21"/>
-<element name="C3" library="capacitor-wima" package="C5B2.5" value="0.1uF" x="3.81" y="-36.83"/>
+<element name="C2" library="capacitor-wima" package="C5B2.5" value="0.1uF" x="31.75" y="10.16"/>
+<element name="C3" library="capacitor-wima" package="C5B2.5" value="0.1uF" x="43.18" y="8.89"/>
+<element name="S3" library="switch" package="TL3XPO" value="TL39PO" x="-31.75" y="3.81"/>
 </elements>
 <signals>
@@
 <wire x1="60.96" y1="35.56" x2="67.31" y2="49.53" width="0" layer="19" extent="1-1"/>
 </signal>
-<signal name="N$10">
-<contactref element="DRIVER1" pad="7"/>
-<contactref element="SV1" pad="4"/>
-<contactref element="MOTOR1" pad="5"/>
-<wire x1="10.16" y1="2.54" x2="19.05" y2="25.4" width="0" layer="19" extent="1-1"/>
-<wire x1="41.91" y1="30.48" x2="10.16" y2="2.54" width="0" layer="19" extent="1-1"/>
-</signal>
-<signal name="N$7">
-<contactref element="DRIVER2" pad="7"/>
-<contactref element="MOTOR2" pad="5"/>
-<contactref element="IMU" pad="1"/>
-<wire x1="62.23" y1="21.59" x2="50.8" y2="35.56" width="0" layer="19" extent="1-1"/>
-<wire x1="17.78" y1="36.83" x2="50.8" y2="35.56" width="0" layer="19" extent="1-1"/>
-</signal>
 <signal name="N$5">
 <contactref element="DRIVER1" pad="4"/>
 <contactref element="SV6" pad="5"/>
-<wire x1="11.43" y1="25.4" x2="11.43" y2="49.53" width="0" layer="19" extent="1-1"/>
+<wire x1="7.62" y1="20.32" x2="11.43" y2="49.53" width="0" layer="19" extent="1-1"/>
 </signal>
 <signal name="N$11">
 <contactref element="SV6" pad="6"/>
 <contactref element="DRIVER2" pad="4"/>
-<wire x1="10.16" y1="36.83" x2="13.97" y2="49.53" width="0" layer="19" extent="1-1"/>
+<wire x1="13.97" y1="36.83" x2="13.97" y2="49.53" width="0" layer="19" extent="1-1"/>
 </signal>
 <signal name="N$2">
@@
 <contactref element="DRIVER1" pad="10"/>
 <contactref element="C2" pad="2"/>
-<wire x1="39.37" y1="30.48" x2="26.67" y2="25.4" width="0" layer="19" extent="1-1"/>
-<wire x1="6.35" y1="-29.21" x2="39.37" y2="30.48" width="0" layer="19" extent="1-1"/>
+<wire x1="39.37" y1="30.48" x2="22.86" y2="20.32" width="0" layer="19" extent="1-1"/>
+<wire x1="34.29" y1="10.16" x2="39.37" y2="30.48" width="0" layer="19" extent="1-1"/>
 </signal>
 <signal name="N$3">
@@
 <contactref element="C3" pad="1"/>
 <contactref element="MOTOR2" pad="3"/>
-<wire x1="57.15" y1="21.59" x2="5.08" y2="36.83" width="0" layer="19" extent="1-1"/>
-<wire x1="1.27" y1="-36.83" x2="57.15" y2="21.59" width="0" layer="19" extent="1-1"/>
+<wire x1="57.15" y1="21.59" x2="8.89" y2="36.83" width="0" layer="19" extent="1-1"/>
+<wire x1="40.64" y1="8.89" x2="57.15" y2="21.59" width="0" layer="19" extent="1-1"/>
 </signal>
 <signal name="N$1">
@@
 <contactref element="DRIVER1" pad="2"/>
 <contactref element="C2" pad="1"/>
-<wire x1="36.83" y1="30.48" x2="6.35" y2="25.4" width="0" layer="19" extent="1-1"/>
-<wire x1="1.27" y1="-29.21" x2="36.83" y2="30.48" width="0" layer="19" extent="1-1"/>
+<wire x1="36.83" y1="30.48" x2="2.54" y2="20.32" width="0" layer="19" extent="1-1"/>
+<wire x1="29.21" y1="10.16" x2="36.83" y2="30.48" width="0" layer="19" extent="1-1"/>
 </signal>
 <signal name="N$6">
@@
 <contactref element="C3" pad="2"/>
 <contactref element="MOTOR2" pad="4"/>
-<wire x1="59.69" y1="21.59" x2="25.4" y2="36.83" width="0" layer="19" extent="1-1"/>
-<wire x1="6.35" y1="-36.83" x2="59.69" y2="21.59" width="0" layer="19" extent="1-1"/>
+<wire x1="59.69" y1="21.59" x2="29.21" y2="36.83" width="0" layer="19" extent="1-1"/>
+<wire x1="45.72" y1="8.89" x2="59.69" y2="21.59" width="0" layer="19" extent="1-1"/>
 </signal>
 <signal name="N$12">
 <contactref element="DRIVER1" pad="5"/>
 <contactref element="SV7" pad="34"/>
-<wire x1="13.97" y1="25.4" x2="87.63" y2="5.08" width="0" layer="19" extent="1-1"/>
+<wire x1="10.16" y1="20.32" x2="87.63" y2="5.08" width="0" layer="19" extent="1-1"/>
 </signal>
 <signal name="N$16">
 <contactref element="DRIVER1" pad="6"/>
 <contactref element="SV7" pad="33"/>
-<wire x1="16.51" y1="25.4" x2="85.09" y2="5.08" width="0" layer="19" extent="1-1"/>
+<wire x1="12.7" y1="20.32" x2="85.09" y2="5.08" width="0" layer="19" extent="1-1"/>
 </signal>
 <signal name="GND">
+<contactref element="X3" pad="1"/>
 <contactref element="MOTOR1" pad="6"/>
-<contactref element="X3" pad="1"/>
 <contactref element="C1" pad="2"/>
 <contactref element="MOTOR2" pad="6"/>
@@
 <contactref element="DRIVER2" pad="1"/>
 <contactref element="IMU" pad="2"/>
-<wire x1="66.04" y1="10.16" x2="71.12" y2="10.43" width="0" layer="19" extent="1-1"/>
-<wire x1="3.81" y1="25.4" x2="66.04" y2="10.16" width="0" layer="19" extent="1-1"/>
-<wire x1="2.54" y1="36.83" x2="3.81" y2="25.4" width="0" layer="19" extent="1-1"/>
-<wire x1="7.62" y1="2.54" x2="3.81" y2="25.4" width="0" layer="19" extent="1-1"/>
-<wire x1="53.34" y1="35.56" x2="7.62" y2="2.54" width="0" layer="19" extent="1-1"/>
 <wire x1="44.45" y1="30.48" x2="53.34" y2="35.56" width="0" layer="19" extent="1-1"/>
-<wire x1="64.77" y1="21.59" x2="44.45" y2="30.48" width="0" layer="19" extent="1-1"/>
+<wire x1="64.77" y1="21.59" x2="53.34" y2="35.56" width="0" layer="19" extent="1-1"/>
+<wire x1="66.04" y1="10.16" x2="64.77" y2="21.59" width="0" layer="19" extent="1-1"/>
+<wire x1="71.12" y1="10.43" x2="66.04" y2="10.16" width="0" layer="19" extent="1-1"/>
+<wire x1="6.35" y1="36.83" x2="44.45" y2="30.48" width="0" layer="19" extent="1-1"/>
+<wire x1="0" y1="20.32" x2="6.35" y2="36.83" width="0" layer="19" extent="1-1"/>
+<wire x1="7.62" y1="2.54" x2="0" y2="20.32" width="0" layer="19" extent="1-1"/>
 </signal>
 <signal name="N$17">
 <contactref element="SV7" pad="32"/>
 <contactref element="DRIVER2" pad="5"/>
-<wire x1="12.7" y1="36.83" x2="87.63" y2="7.62" width="0" layer="19" extent="1-1"/>
+<wire x1="16.51" y1="36.83" x2="87.63" y2="7.62" width="0" layer="19" extent="1-1"/>
 </signal>
 <signal name="N$18">
 <contactref element="DRIVER2" pad="6"/>
 <contactref element="SV7" pad="31"/>
-<wire x1="15.24" y1="36.83" x2="85.09" y2="7.62" width="0" layer="19" extent="1-1"/>
+<wire x1="19.05" y1="36.83" x2="85.09" y2="7.62" width="0" layer="19" extent="1-1"/>
 </signal>
 <signal name="VCC">
+<contactref element="X3" pad="2"/>
+<contactref element="S3" pad="2"/>
+<wire x1="-31.75" y1="3.81" x2="71.12" y2="12.43" width="0" layer="19" extent="1-1"/>
+</signal>
+<signal name="N$7">
+<contactref element="MOTOR1" pad="5"/>
+<contactref element="MOTOR2" pad="5"/>
+<contactref element="DRIVER1" pad="7"/>
+<contactref element="SV1" pad="4"/>
+<contactref element="DRIVER2" pad="7"/>
+<contactref element="IMU" pad="1"/>
+<wire x1="41.91" y1="30.48" x2="50.8" y2="35.56" width="0" layer="19" extent="1-1"/>
+<wire x1="62.23" y1="21.59" x2="50.8" y2="35.56" width="0" layer="19" extent="1-1"/>
+<wire x1="15.24" y1="20.32" x2="41.91" y2="30.48" width="0" layer="19" extent="1-1"/>
+<wire x1="21.59" y1="36.83" x2="15.24" y2="20.32" width="0" layer="19" extent="1-1"/>
+<wire x1="10.16" y1="2.54" x2="15.24" y2="20.32" width="0" layer="19" extent="1-1"/>
+</signal>
+<signal name="N$10">
+<contactref element="C1" pad="1"/>
+<contactref element="SV1" pad="1"/>
+<contactref element="DRIVER2" pad="8"/>
 <contactref element="DRIVER1" pad="8"/>
-<contactref element="X3" pad="2"/>
-<contactref element="C1" pad="1"/>
-<contactref element="DRIVER2" pad="8"/>
-<contactref element="SV1" pad="1"/>
-<wire x1="60.96" y1="10.16" x2="71.12" y2="12.43" width="0" layer="19" extent="1-1"/>
-<wire x1="21.59" y1="25.4" x2="60.96" y2="10.16" width="0" layer="19" extent="1-1"/>
-<wire x1="20.32" y1="36.83" x2="21.59" y2="25.4" width="0" layer="19" extent="1-1"/>
-<wire x1="2.54" y1="2.54" x2="21.59" y2="25.4" width="0" layer="19" extent="1-1"/>
+<contactref element="S3" pad="1"/>
+<wire x1="17.78" y1="20.32" x2="60.96" y2="10.16" width="0" layer="19" extent="1-1"/>
+<wire x1="24.13" y1="36.83" x2="17.78" y2="20.32" width="0" layer="19" extent="1-1"/>
+<wire x1="2.54" y1="2.54" x2="17.78" y2="20.32" width="0" layer="19" extent="1-1"/>
+<wire x1="-34.29" y1="3.81" x2="2.54" y2="2.54" width="0" layer="19" extent="1-1"/>
 </signal>
 </signals>
