File: circuit/eagle/projects/Inverted_Pendulum-in-TAHU/untitled2.brd (EAGLE design)
At the start: 17 parts, among them X3 332-02

Commit message: add 回路の完成形＆スライド
Parts:
- added VS-C3: (no value), con-lstb:MA05-2
- moved S3 98.0 mm to (59.1, 40.6), turned to 90 degrees
- moved DRIVER1 49.1 mm to (60.3, 24.6)
- moved DRIVER2 48.3 mm to (60.3, 13.9)
- moved MOTOR2 30.9 mm to (27.9, 16.5), turned to 90 degrees
- moved X3 28.8 mm to (67.3, 40.0), turned to 180 degrees
- moved C1 28.2 mm to (74.3, 36.2), turned to 90 degrees
- moved C2 26.9 mm to (22.9, 35.6), turned to 90 degrees
- moved IMU 25.5 mm to (80.0, 43.8), turned to 180 degrees
- moved SV1 25.4 mm to (36.8, 2.54), turned to 180 degrees
- moved SV2 22.9 mm to (59.7, 2.54), turned to 180 degrees
- moved C3 21.3 mm to (22.9, 15.2), turned to 90 degrees
- moved SV3 20.4 mm to (82.5, 2.54), turned to 180 degrees
- moved SV6 16.5 mm to (29.2, 49.5)
- moved SV5 15.2 mm to (54.6, 49.5)
- moved SV4 14.0 mm to (77.5, 49.5)
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Connections:
- new net N$22: SV5.3, VS-C3.5
- new net N$23: SV6.1, VS-C3.6
- new net N$24: DRIVER1.4, SV7.12
- net GND: now also VS-C3.10
- net N$11: now also SV7.10; no longer SV6.6
- net N$12: now also SV7.16; no longer SV7.34
- net N$13: now also MOTOR1.1; no longer MOTOR2.1, SV6.8
- net N$14: now also SV7.26; no longer SV7.29
- net N$15: now also SV7.24; no longer SV7.30
- net N$16: now also SV7.14; no longer SV7.33
- net N$17: now also SV7.8; no longer SV7.32
- net N$18: now also SV7.6; no longer SV7.31
- net N$19: now also SV1.5, VS-C3.9; no longer SV5.1, SV6.4
- net N$20: now also SV6.5, VS-C3.3; no longer SV5.4, SV6.7
- net N$21: now also SV6.6, VS-C3.4; no longer SV5.7, SV6.10
- net N$5: now also IMU.1, SV7.36; no longer DRIVER1.4, SV6.5
- net N$6: now also MOTOR2.1; no longer MOTOR1.1, SV6.9
- net N$7: no longer IMU.1
Other:
- board outline added: 100 x 53 mm
